File: hardware/in.kicad_sch (KiCad schematic)
At the start: 1 part, among them J62 Screw_Terminal_01x04

Commit message: added translations
Changed lines of the file:
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@@
 	(generator_version "8.0")
 	(paper "A4")
-	(junction
-		(at 135.89 106.68)
-		(diameter 0)
-		(color 0 0 0 0)
-	)
-	(junction
-		(at 130.81 104.14)
-		(diameter 0)
-		(color 0 0 0 0)
-	)
 	(bus_entry
 		(at 129.54 123.19)
@@
 	(wire
 		(pts
-			(xy 130.81 102.87) (xy 130.81 104.14)
-		)
-		(stroke
-			(width 0)
-			(type default)
-		)
-	)
-	(wire
-		(pts
 			(xy 130.81 104.14) (xy 130.81 109.22)
 		)
@@
 		)
 	)
-	(wire
-		(pts
-			(xy 135.89 106.68) (xy 144.78 106.68)
-		)
-		(stroke
-			(width 0)
-			(type default)
-		)
-	)
 	(bus
 		(pts
@@
 		(pts
 			(xy 116.84 106.68) (xy 135.89 106.68)
-		)
-		(stroke
-			(width 0)
-			(type default)
-		)
-	)
-	(wire
-		(pts
-			(xy 144.78 106.68) (xy 144.78 102.87)
 		)
 		(stroke
@@
 			)
 			(justify left)
-		)
-	)
-	(symbol
-		(lib_id "power:PWR_FLAG")
-		(at 144.78 102.87 0)
-		(unit 1)
-		(exclude_from_sim no)
-		(in_bom yes)
-		(on_board yes)
-		(dnp no)
-		(property "Reference" "#FLG0301"
-			(at 144.78 100.965 0)
-			(effects
-				(font
-					(size 1.27 1.27)
-				)
-				(hide yes)
-			)
-		)
-		(property "Value" "PWR_FLAG"
-			(at 144.78 99.06 0)
-			(effects
-				(font
-					(size 1.27 1.27)
-				)
-			)
-		)
-		(property "Footprint" ""
-			(at 144.78 102.87 0)
-			(effects
-				(font
-					(size 1.27 1.27)
-				)
-				(hide yes)
-			)
-		)
-		(property "Datasheet" "~"
-			(at 144.78 102.87 0)
-			(effects
-				(font
-					(size 1.27 1.27)
-				)
-				(hide yes)
-			)
-		)
-		(property "Description" ""
-			(at 144.78 102.87 0)
-			(effects
-				(font
-					(size 1.27 1.27)
-				)
-				(hide yes)
-			)
-		)
-		(pin "1"
-		)
-		(instances
-			(project "oneFit"
-				(path "/5298ac75-044e-4260-bbaf-3f2b608479b0/51c5c96b-4881-4f86-93e6-5d523794193d"
-					(reference "#FLG0301")
-					(unit 1)
-				)
-			)
 		)
 	)
@@
 		(dnp no)
 		(fields_autoplaced yes)
-		(property "Reference" "#PWR0302"
+		(property "Reference" "#PWR0702"
 			(at 130.81 115.57 0)
 			(effects
@@
 		)
 		(instances
-			(project "oneFit"
+			(project ""
 				(path "/5298ac75-044e-4260-bbaf-3f2b608479b0/51c5c96b-4881-4f86-93e6-5d523794193d"
-					(reference "#PWR0302")
+					(reference "#PWR0702")
 					(unit 1)
 				)
@@
 		(on_board yes)
 		(dnp no)
-		(property "Reference" "#PWR0301"
+		(property "Reference" "#PWR0703"
 			(at 135.89 106.68 0)
 			(effects
@@
 		)
 		(instances
-			(project "oneFit"
+			(project ""
 				(path "/5298ac75-044e-4260-bbaf-3f2b608479b0/51c5c96b-4881-4f86-93e6-5d523794193d"
-					(reference "#PWR0301")
-					(unit 1)
-				)
-			)
-		)
-	)
-	(symbol
-		(lib_id "power:PWR_FLAG")
-		(at 130.81 102.87 0)
-		(unit 1)
-		(exclude_from_sim no)
-		(in_bom yes)
-		(on_board yes)
-		(dnp no)
-		(property "Reference" "#FLG0302"
-			(at 130.81 100.965 0)
-			(effects
-				(font
-					(size 1.27 1.27)
-				)
-				(hide yes)
-			)
-		)
-		(property "Value" "PWR_FLAG"
-			(at 127 99.06 0)
-			(effects
-				(font
-					(size 1.27 1.27)
-				)
-			)
-		)
-		(property "Footprint" ""
-			(at 130.81 102.87 0)
-			(effects
-				(font
-					(size 1.27 1.27)
-				)
-				(hide yes)
-			)
-		)
-		(property "Datasheet" "~"
-			(at 130.81 102.87 0)
-			(effects
-				(font
-					(size 1.27 1.27)
-				)
-				(hide yes)
-			)
-		)
-		(property "Description" ""
-			(at 130.81 102.87 0)
-			(effects
-				(font
-					(size 1.27 1.27)
-				)
-				(hide yes)
-			)
-		)
-		(pin "1"
-		)
-		(instances
-			(project "oneFit"
-				(path "/5298ac75-044e-4260-bbaf-3f2b608479b0/51c5c96b-4881-4f86-93e6-5d523794193d"
-					(reference "#FLG0302")
+					(reference "#PWR0703")
 					(unit 1)
 				)
@@
 		)
 		(instances
-			(project "oneFit"
+			(project ""
 				(path "/5298ac75-044e-4260-bbaf-3f2b608479b0/51c5c96b-4881-4f86-93e6-5d523794193d"
 					(reference "J62")
